File: Production Files/Micro_SD_Block_GiantPanel_v20.brd (EAGLE design)
At the start: 274.8 x 206.8 mm, 472 parts, among them U1 USD-SOCKETNEW, U10 EDISON_CONNECTOR_FULLHEADER, U100 TXB0108, U101 EDISON_CONNECTOR_FULLMOUNTING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, U102 EDISON_CONNECTOR_FULLHEADER, U103 USD-SOCKETNEW, U104 TXB0108, U105 EDISON_CONNECTOR_FULLMOUNTING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, U106 EDISON_CONNECTOR_FULLHEADER, U107 USD-SOCKETNEW, U108 TXB0108, U109 EDISON_CONNECTOR_FULLMOUNTING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, U11 USD-SOCKETNEW, U110 EDISON_CONNECTOR_FULLHEADER, U111 USD-SOCKETNEW, U112 TXB0108, U113 EDISON_CONNECTOR_FULLMOUNTING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, U114 EDISON_CONNECTOR_FULLHEADER, U115 USD-SOCKETNEW, U116 TXB0108, U117 EDISON_CONNECTOR_FULLMOUNTING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, U118 EDISON_CONNECTOR_FULLHEADER, U119 USD-SOCKETNEW, U12 TXB0108, U120 TXB0108, U121 EDISON_CONNECTOR_FULLMOUNTING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, U122 EDISON_CONNECTOR_FULLHEADER, U123 USD-SOCKETNEW, U124 TXB0108, U125 EDISON_CONNECTOR_FULLMOUNTING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, U126 EDISON_CONNECTOR_FULLHEADER, U127 USD-SOCKETNEW, U128 TXB0108, U13 EDISON_CONNECTOR_FULLMOUNTING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, U14 EDISON_CONNECTOR_FULLHEADER, U15 USD-SOCKETNEW, U16 TXB0108, U17 EDISON_CONNECTOR_FULLMOUNTING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, U18 EDISON_CONNECTOR_FULLHEADER, U19 USD-SOCKETNEW, U2 EDISON_CONNECTOR_FULLMOUNTING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, U20 TXB0108, U21 EDISON_CONNECTOR_FULLMOUNTING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, U22 EDISON_CONNECTOR_FULLHEADER, U23 USD-SOCKETNEW, U24 TXB0108, U25 EDISON_CONNECTOR_FULLMOUNTING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, U26 EDISON_CONNECTOR_FULLHEADER, U27 USD-SOCKETNEW, U28 TXB0108, U29 EDISON_CONNECTOR_FULLMOUNTING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, U3 EDISON_CONNECTOR_FULLHEADER, U30 EDISON_CONNECTOR_FULLHEADER, U31 USD-SOCKETNEW, U32 TXB0108, U33 EDISON_CONNECTOR_FULLMOUNTING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, U34 EDISON_CONNECTOR_FULLHEADER, U35 USD-SOCKETNEW, U36 TXB0108, U37 EDISON_CONNECTOR_FULLMOUNTING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, U38 EDISON_CONNECTOR_FULLHEADER, U39 USD-SOCKETNEW, U4 TXB0108, U40 TXB0108, U41 EDISON_CONNECTOR_FULLMOUNTING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, U42 EDISON_CONNECTOR_FULLHEADER, U43 USD-SOCKETNEW, U44 TXB0108, U45 EDISON_CONNECTOR_FULLMOUNTING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, U46 EDISON_CONNECTOR_FULLHEADER, U47 USD-SOCKETNEW, U48 TXB0108, U49 EDISON_CONNECTOR_FULLMOUNTING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, U5 EDISON_CONNECTOR_FULLMOUNTING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, U50 EDISON_CONNECTOR_FULLHEADER, U51 USD-SOCKETNEW, U52 TXB0108, U53 EDISON_CONNECTOR_FULLMOUNTING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, U54 EDISON_CONNECTOR_FULLHEADER, U55 USD-SOCKETNEW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

Commit message: removed v10 panels and created v20 panels
Connections:
- net GND: no longer U1.CD2
- net GND1: no longer U7.CD2
- net GND10: no longer U43.CD2
- net GND11: no longer U47.CD2
- net GND12: no longer U51.CD2
- net GND13: no longer U55.CD2
- net GND14: no longer U59.CD2
- net GND15: no longer U63.CD2
- net GND16: no longer U67.CD2
- net GND17: no longer U71.CD2
- net GND18: no longer U75.CD2
- net GND19: no longer U79.CD2
- net GND2: no longer U11.CD2
- net GND20: no longer U83.CD2
- net GND21: no longer U87.CD2
- net GND22: no longer U91.CD2
- net GND23: no longer U95.CD2
- net GND24: no longer U99.CD2
- net GND25: no longer U103.CD2
- net GND26: no longer U107.CD2
- net GND27: no longer U111.CD2
- net GND28: no longer U115.CD2
- net GND29: no longer U119.CD2
- net GND3: no longer U15.CD2
- net GND30: no longer U123.CD2
- net GND31: no longer U127.CD2
- net GND4: no longer U19.CD2
- net GND5: no longer U23.CD2
- net GND6: no longer U27.CD2
- net GND7: no longer U31.CD2
- net GND8: no longer U35.CD2
- net GND9: no longer U39.CD2
Other:
- board text added: "v20"
- board text removed: "v10"
